Commit message: Clarify where effort can be changed

File: SpiderBot/spider.urdf (robot description, URDF)
Before this commit: robot blocky_spider, 31 links, 30 joints
Joints:
- joint joint_body_leg_hip_0: limit lower=-0.9599310885968813 upper=0.9599310885968813 effort=25 velocity=4.0 -> lower=-0.9599310885968813 upper=0.9599310885968813 effort=0.25 velocity=4.0
- joint joint_body_leg_hip_1: limit lower=-0.9599310885968813 upper=0.9599310885968813 effort=25 velocity=4.0 -> lower=-0.9599310885968813 upper=0.9599310885968813 effort=0.25 velocity=4.0
- joint joint_body_leg_hip_2: limit lower=-0.9599310885968813 upper=0.9599310885968813 effort=25 velocity=4.0 -> lower=-0.9599310885968813 upper=0.9599310885968813 effort=0.25 velocity=4.0
- joint joint_body_leg_hip_3: limit lower=-0.9599310885968813 upper=0.9599310885968813 effort=25 velocity=4.0 -> lower=-0.9599310885968813 upper=0.9599310885968813 effort=0.25 velocity=4.0
- joint joint_body_leg_hip_4: limit lower=-0.9599310885968813 upper=0.9599310885968813 effort=25 velocity=4.0 -> lower=-0.9599310885968813 upper=0.9599310885968813 effort=0.25 velocity=4.0
- joint joint_body_leg_hip_5: limit lower=-0.9599310885968813 upper=0.9599310885968813 effort=25 velocity=4.0 -> lower=-0.9599310885968813 upper=0.9599310885968813 effort=0.25 velocity=4.0
- joint joint_leg_hip_leg_upper_0: limit lower=-1.3089969389957472 upper=1.3089969389957472 effort=12 velocity=5.0 -> lower=-1.3089969389957472 upper=1.3089969389957472 effort=0.12 velocity=5.0
- joint joint_leg_hip_leg_upper_1: limit lower=-1.3089969389957472 upper=1.3089969389957472 effort=12 velocity=5.0 -> lower=-1.3089969389957472 upper=1.3089969389957472 effort=0.12 velocity=5.0
- joint joint_leg_hip_leg_upper_2: limit lower=-1.3089969389957472 upper=1.3089969389957472 effort=12 velocity=5.0 -> lower=-1.3089969389957472 upper=1.3089969389957472 effort=0.12 velocity=5.0
- joint joint_leg_hip_leg_upper_3: limit lower=-1.3089969389957472 upper=1.3089969389957472 effort=12 velocity=5.0 -> lower=-1.3089969389957472 upper=1.3089969389957472 effort=0.12 velocity=5.0
- joint joint_leg_hip_leg_upper_4: limit lower=-1.3089969389957472 upper=1.3089969389957472 effort=12 velocity=5.0 -> lower=-1.3089969389957472 upper=1.3089969389957472 effort=0.12 velocity=5.0
- joint joint_leg_hip_leg_upper_5: limit lower=-1.3089969389957472 upper=1.3089969389957472 effort=12 velocity=5.0 -> lower=-1.3089969389957472 upper=1.3089969389957472 effort=0.12 velocity=5.0
- joint joint_leg_middle_leg_lower_0: limit lower=-1.5707963267948966 upper=0.7853981633974483 effort=4 velocity=8.0 -> lower=-1.5707963267948966 upper=0.7853981633974483 effort=0.04 velocity=8.0
- joint joint_leg_middle_leg_lower_1: limit lower=-1.5707963267948966 upper=0.7853981633974483 effort=4 velocity=8.0 -> lower=-1.5707963267948966 upper=0.7853981633974483 effort=0.04 velocity=8.0
- joint joint_leg_middle_leg_lower_2: limit lower=-1.5707963267948966 upper=0.7853981633974483 effort=4 velocity=8.0 -> lower=-1.5707963267948966 upper=0.7853981633974483 effort=0.04 velocity=8.0
- joint joint_leg_middle_leg_lower_3: limit lower=-1.5707963267948966 upper=0.7853981633974483 effort=4 velocity=8.0 -> lower=-1.5707963267948966 upper=0.7853981633974483 effort=0.04 velocity=8.0
- joint joint_leg_middle_leg_lower_4: limit lower=-1.5707963267948966 upper=0.7853981633974483 effort=4 velocity=8.0 -> lower=-1.5707963267948966 upper=0.7853981633974483 effort=0.04 velocity=8.0
- joint joint_leg_middle_leg_lower_5: limit lower=-1.5707963267948966 upper=0.7853981633974483 effort=4 velocity=8.0 -> lower=-1.5707963267948966 upper=0.7853981633974483 effort=0.04 velocity=8.0
- joint joint_leg_upper_leg_middle_0: limit lower=-1.5707963267948966 upper=0.3490658503988659 effort=8 velocity=6.0 -> lower=-1.5707963267948966 upper=0.3490658503988659 effort=0.08 velocity=6.0
- joint joint_leg_upper_leg_middle_1: limit lower=-1.5707963267948966 upper=0.3490658503988659 effort=8 velocity=6.0 -> lower=-1.5707963267948966 upper=0.3490658503988659 effort=0.08 velocity=6.0
- joint joint_leg_upper_leg_middle_2: limit lower=-1.5707963267948966 upper=0.3490658503988659 effort=8 velocity=6.0 -> lower=-1.5707963267948966 upper=0.3490658503988659 effort=0.08 velocity=6.0
- joint joint_leg_upper_leg_middle_3: limit lower=-1.5707963267948966 upper=0.3490658503988659 effort=8 velocity=6.0 -> lower=-1.5707963267948966 upper=0.3490658503988659 effort=0.08 velocity=6.0
- joint joint_leg_upper_leg_middle_4: limit lower=-1.5707963267948966 upper=0.3490658503988659 effort=8 velocity=6.0 -> lower=-1.5707963267948966 upper=0.3490658503988659 effort=0.08 velocity=6.0
- joint joint_leg_upper_leg_middle_5: limit lower=-1.5707963267948966 upper=0.3490658503988659 effort=8 velocity=6.0 -> lower=-1.5707963267948966 upper=0.3490658503988659 effort=0.08 velocity=6.0

Commit message: tweaks to config

File: SpiderBot/spider.urdf (robot description, URDF)
Before this commit: robot blocky_spider, 31 links, 30 joints
Joints:
- joint joint_body_leg_hip_0: limit lower=-0.9599310885968813 upper=0.9599310885968813 effort=0.25 velocity=4.0 -> lower=-0.9599310885968813 upper=0.9599310885968813 effort=25 velocity=4.0
- joint joint_body_leg_hip_1: limit lower=-0.9599310885968813 upper=0.9599310885968813 effort=0.25 velocity=4.0 -> lower=-0.9599310885968813 upper=0.9599310885968813 effort=25 velocity=4.0
- joint joint_body_leg_hip_2: limit lower=-0.9599310885968813 upper=0.9599310885968813 effort=0.25 velocity=4.0 -> lower=-0.9599310885968813 upper=0.9599310885968813 effort=25 velocity=4.0
- joint joint_body_leg_hip_3: limit lower=-0.9599310885968813 upper=0.9599310885968813 effort=0.25 velocity=4.0 -> lower=-0.9599310885968813 upper=0.9599310885968813 effort=25 velocity=4.0
- joint joint_body_leg_hip_4: limit lower=-0.9599310885968813 upper=0.9599310885968813 effort=0.25 velocity=4.0 -> lower=-0.9599310885968813 upper=0.9599310885968813 effort=25 velocity=4.0
- joint joint_body_leg_hip_5: limit lower=-0.9599310885968813 upper=0.9599310885968813 effort=0.25 velocity=4.0 -> lower=-0.9599310885968813 upper=0.9599310885968813 effort=25 velocity=4.0
- joint joint_leg_hip_leg_upper_0: limit lower=-1.3089969389957472 upper=1.3089969389957472 effort=0.12 velocity=5.0 -> lower=-1.3089969389957472 upper=1.3089969389957472 effort=12 velocity=5.0
- joint joint_leg_hip_leg_upper_1: limit lower=-1.3089969389957472 upper=1.3089969389957472 effort=0.12 velocity=5.0 -> lower=-1.3089969389957472 upper=1.3089969389957472 effort=12 velocity=5.0
- joint joint_leg_hip_leg_upper_2: limit lower=-1.3089969389957472 upper=1.3089969389957472 effort=0.12 velocity=5.0 -> lower=-1.3089969389957472 upper=1.3089969389957472 effort=12 velocity=5.0
- joint joint_leg_hip_leg_upper_3: limit lower=-1.3089969389957472 upper=1.3089969389957472 effort=0.12 velocity=5.0 -> lower=-1.3089969389957472 upper=1.3089969389957472 effort=12 velocity=5.0
- joint joint_leg_hip_leg_upper_4: limit lower=-1.3089969389957472 upper=1.3089969389957472 effort=0.12 velocity=5.0 -> lower=-1.3089969389957472 upper=1.3089969389957472 effort=12 velocity=5.0
- joint joint_leg_hip_leg_upper_5: limit lower=-1.3089969389957472 upper=1.3089969389957472 effort=0.12 velocity=5.0 -> lower=-1.3089969389957472 upper=1.3089969389957472 effort=12 velocity=5.0
- joint joint_leg_middle_leg_lower_0: limit lower=-1.5707963267948966 upper=0.7853981633974483 effort=0.04 velocity=8.0 -> lower=-1.5707963267948966 upper=0.7853981633974483 effort=4 velocity=8.0
- joint joint_leg_middle_leg_lower_1: limit lower=-1.5707963267948966 upper=0.7853981633974483 effort=0.04 velocity=8.0 -> lower=-1.5707963267948966 upper=0.7853981633974483 effort=4 velocity=8.0
- joint joint_leg_middle_leg_lower_2: limit lower=-1.5707963267948966 upper=0.7853981633974483 effort=0.04 velocity=8.0 -> lower=-1.5707963267948966 upper=0.7853981633974483 effort=4 velocity=8.0
- joint joint_leg_middle_leg_lower_3: limit lower=-1.5707963267948966 upper=0.7853981633974483 effort=0.04 velocity=8.0 -> lower=-1.5707963267948966 upper=0.7853981633974483 effort=4 velocity=8.0
- joint joint_leg_middle_leg_lower_4: limit lower=-1.5707963267948966 upper=0.7853981633974483 effort=0.04 velocity=8.0 -> lower=-1.5707963267948966 upper=0.7853981633974483 effort=4 velocity=8.0
- joint joint_leg_middle_leg_lower_5: limit lower=-1.5707963267948966 upper=0.7853981633974483 effort=0.04 velocity=8.0 -> lower=-1.5707963267948966 upper=0.7853981633974483 effort=4 velocity=8.0
- joint joint_leg_upper_leg_middle_0: limit lower=-1.5707963267948966 upper=0.3490658503988659 effort=0.08 velocity=6.0 -> lower=-1.5707963267948966 upper=0.3490658503988659 effort=8 velocity=6.0
- joint joint_leg_upper_leg_middle_1: limit lower=-1.5707963267948966 upper=0.3490658503988659 effort=0.08 velocity=6.0 -> lower=-1.5707963267948966 upper=0.3490658503988659 effort=8 velocity=6.0
- joint joint_leg_upper_leg_middle_2: limit lower=-1.5707963267948966 upper=0.3490658503988659 effort=0.08 velocity=6.0 -> lower=-1.5707963267948966 upper=0.3490658503988659 effort=8 velocity=6.0
- joint joint_leg_upper_leg_middle_3: limit lower=-1.5707963267948966 upper=0.3490658503988659 effort=0.08 velocity=6.0 -> lower=-1.5707963267948966 upper=0.3490658503988659 effort=8 velocity=6.0
- joint joint_leg_upper_leg_middle_4: limit lower=-1.5707963267948966 upper=0.3490658503988659 effort=0.08 velocity=6.0 -> lower=-1.5707963267948966 upper=0.3490658503988659 effort=8 velocity=6.0
- joint joint_leg_upper_leg_middle_5: limit lower=-1.5707963267948966 upper=0.3490658503988659 effort=0.08 velocity=6.0 -> lower=-1.5707963267948966 upper=0.3490658503988659 effort=8 velocity=6.0

Commit message: Updated with fixed joint values

File: SpiderBot/spider.urdf (robot description, URDF)
Before this commit: robot blocky_spider, 31 links, 30 joints
Joints:
- joint joint_body_leg_hip_0: limit lower=-0.9599310885968813 upper=0.9599310885968813 effort=25 velocity=4.0 -> lower=-0.9599310885968813 upper=0.9599310885968813 effort=12 velocity=12.0
- joint joint_body_leg_hip_1: limit lower=-0.9599310885968813 upper=0.9599310885968813 effort=25 velocity=4.0 -> lower=-0.9599310885968813 upper=0.9599310885968813 effort=12 velocity=12.0
- joint joint_body_leg_hip_2: limit lower=-0.9599310885968813 upper=0.9599310885968813 effort=25 velocity=4.0 -> lower=-0.9599310885968813 upper=0.9599310885968813 effort=12 velocity=12.0
- joint joint_body_leg_hip_3: limit lower=-0.9599310885968813 upper=0.9599310885968813 effort=25 velocity=4.0 -> lower=-0.9599310885968813 upper=0.9599310885968813 effort=12 velocity=12.0
- joint joint_body_leg_hip_4: limit lower=-0.9599310885968813 upper=0.9599310885968813 effort=25 velocity=4.0 -> lower=-0.9599310885968813 upper=0.9599310885968813 effort=12 velocity=12.0
- joint joint_body_leg_hip_5: limit lower=-0.9599310885968813 upper=0.9599310885968813 effort=25 velocity=4.0 -> lower=-0.9599310885968813 upper=0.9599310885968813 effort=12 velocity=12.0
- joint joint_leg_hip_leg_upper_0: limit lower=-1.3089969389957472 upper=1.3089969389957472 effort=12 velocity=5.0 -> lower=-1.3089969389957472 upper=1.3089969389957472 effort=30 velocity=15.0
- joint joint_leg_hip_leg_upper_1: limit lower=-1.3089969389957472 upper=1.3089969389957472 effort=12 velocity=5.0 -> lower=-1.3089969389957472 upper=1.3089969389957472 effort=30 velocity=15.0
- joint joint_leg_hip_leg_upper_2: limit lower=-1.3089969389957472 upper=1.3089969389957472 effort=12 velocity=5.0 -> lower=-1.3089969389957472 upper=1.3089969389957472 effort=30 velocity=15.0
- joint joint_leg_hip_leg_upper_3: limit lower=-1.3089969389957472 upper=1.3089969389957472 effort=12 velocity=5.0 -> lower=-1.3089969389957472 upper=1.3089969389957472 effort=30 velocity=15.0
- joint joint_leg_hip_leg_upper_4: limit lower=-1.3089969389957472 upper=1.3089969389957472 effort=12 velocity=5.0 -> lower=-1.3089969389957472 upper=1.3089969389957472 effort=30 velocity=15.0
- joint joint_leg_hip_leg_upper_5: limit lower=-1.3089969389957472 upper=1.3089969389957472 effort=12 velocity=5.0 -> lower=-1.3089969389957472 upper=1.3089969389957472 effort=30 velocity=15.0
- joint joint_leg_middle_leg_lower_0: limit lower=-1.5707963267948966 upper=0.7853981633974483 effort=4 velocity=8.0 -> lower=-1.5707963267948966 upper=0.7853981633974483 effort=11 velocity=15.0
- joint joint_leg_middle_leg_lower_1: limit lower=-1.5707963267948966 upper=0.7853981633974483 effort=4 velocity=8.0 -> lower=-1.5707963267948966 upper=0.7853981633974483 effort=11 velocity=15.0
- joint joint_leg_middle_leg_lower_2: limit lower=-1.5707963267948966 upper=0.7853981633974483 effort=4 velocity=8.0 -> lower=-1.5707963267948966 upper=0.7853981633974483 effort=11 velocity=15.0
- joint joint_leg_middle_leg_lower_3: limit lower=-1.5707963267948966 upper=0.7853981633974483 effort=4 velocity=8.0 -> lower=-1.5707963267948966 upper=0.7853981633974483 effort=11 velocity=15.0
- joint joint_leg_middle_leg_lower_4: limit lower=-1.5707963267948966 upper=0.7853981633974483 effort=4 velocity=8.0 -> lower=-1.5707963267948966 upper=0.7853981633974483 effort=11 velocity=15.0
- joint joint_leg_middle_leg_lower_5: limit lower=-1.5707963267948966 upper=0.7853981633974483 effort=4 velocity=8.0 -> lower=-1.5707963267948966 upper=0.7853981633974483 effort=11 velocity=15.0
- joint joint_leg_upper_leg_middle_0: limit lower=-1.5707963267948966 upper=0.3490658503988659 effort=8 velocity=6.0 -> lower=-1.5707963267948966 upper=0.3490658503988659 effort=22 velocity=15.0
- joint joint_leg_upper_leg_middle_1: limit lower=-1.5707963267948966 upper=0.3490658503988659 effort=8 velocity=6.0 -> lower=-1.5707963267948966 upper=0.3490658503988659 effort=22 velocity=15.0
- joint joint_leg_upper_leg_middle_2: limit lower=-1.5707963267948966 upper=0.3490658503988659 effort=8 velocity=6.0 -> lower=-1.5707963267948966 upper=0.3490658503988659 effort=22 velocity=15.0
- joint joint_leg_upper_leg_middle_3: limit lower=-1.5707963267948966 upper=0.3490658503988659 effort=8 velocity=6.0 -> lower=-1.5707963267948966 upper=0.3490658503988659 effort=22 velocity=15.0
- joint joint_leg_upper_leg_middle_4: limit lower=-1.5707963267948966 upper=0.3490658503988659 effort=8 velocity=6.0 -> lower=-1.5707963267948966 upper=0.3490658503988659 effort=22 velocity=15.0
- joint joint_leg_upper_leg_middle_5: limit lower=-1.5707963267948966 upper=0.3490658503988659 effort=8 velocity=6.0 -> lower=-1.5707963267948966 upper=0.3490658503988659 effort=22 velocity=15.0

Commit message: new everything

File: SpiderBot/spider.urdf (robot description, URDF)
Before this commit: robot blocky_spider, 31 links, 30 joints
Links:
- link body: mass 9.019807 -> 21.991149; geometry collision cylinder length=0.025 radius=0.2; visual cylinder length=0.025 radius=0.2
- link leg_foot_0: mass 0.027768 -> 0.000000
- link leg_foot_1: mass 0.027768 -> 0.000000
- link leg_foot_2: mass 0.027768 -> 0.000000
- link leg_foot_3: mass 0.027768 -> 0.000000
- link leg_foot_4: mass 0.027768 -> 0.000000
- link leg_foot_5: mass 0.027768 -> 0.000000
- link leg_hip_0: mass 0.018750 -> 0.109375
- link leg_hip_1: mass 0.018750 -> 0.109375
- link leg_hip_2: mass 0.018750 -> 0.109375
- link leg_hip_3: mass 0.018750 -> 0.109375
- link leg_hip_4: mass 0.018750 -> 0.109375
- link leg_hip_5: mass 0.018750 -> 0.109375
- link leg_lower_0: mass 0.131250 -> 0.765625
- link leg_lower_1: mass 0.131250 -> 0.765625
- link leg_lower_2: mass 0.131250 -> 0.765625
- link leg_lower_3: mass 0.131250 -> 0.765625
- link leg_lower_4: mass 0.131250 -> 0.765625
- link leg_lower_5: mass 0.131250 -> 0.765625
- link leg_middle_0: mass 0.131250 -> 0.765625
- link leg_middle_1: mass 0.131250 -> 0.765625
- link leg_middle_2: mass 0.131250 -> 0.765625
- link leg_middle_3: mass 0.131250 -> 0.765625
- link leg_middle_4: mass 0.131250 -> 0.765625
- link leg_middle_5: mass 0.131250 -> 0.765625
- link leg_upper_0: mass 0.093750 -> 0.546875
- link leg_upper_1: mass 0.093750 -> 0.546875
- link leg_upper_2: mass 0.093750 -> 0.546875
- link leg_upper_3: mass 0.093750 -> 0.546875
- link leg_upper_4: mass 0.093750 -> 0.546875
- link leg_upper_5: mass 0.093750 -> 0.546875
Joints:
- joint joint_body_leg_hip_0: limit lower=-0.9599310885968813 upper=0.9599310885968813 effort=12 velocity=12.0 -> lower=-0.7853981633974483 upper=0.7853981633974483 effort=45; origin xyz=0.21875 0.0 0 rpy=0 0 0.0 -> xyz=0.2 0.0 0 rpy=0 0 0.0
- joint joint_body_leg_hip_1: limit lower=-0.9599310885968813 upper=0.9599310885968813 effort=12 velocity=12.0 -> lower=-0.7853981633974483 upper=0.7853981633974483 effort=45; origin xyz=0.10937500000000003 0.18944305707784595 0 rpy=0 0 1.0471975511965976 -> xyz=0.10000000000000003 0.17320508075688773 0 rpy=0 0 1.0471975511965976
- joint joint_body_leg_hip_2: limit lower=-0.9599310885968813 upper=0.9599310885968813 effort=12 velocity=12.0 -> lower=-0.7853981633974483 upper=0.7853981633974483 effort=45; origin xyz=-0.10937499999999994 0.18944305707784598 0 rpy=0 0 2.0943951023931953 -> xyz=-0.09999999999999996 0.17320508075688776 0 rpy=0 0 2.0943951023931953
- joint joint_body_leg_hip_3: limit lower=-0.9599310885968813 upper=0.9599310885968813 effort=12 velocity=12.0 -> lower=-0.7853981633974483 upper=0.7853981633974483 effort=45; origin xyz=-0.21875 2.678914873134835e-17 0 rpy=0 0 3.141592653589793 -> xyz=-0.2 2.4492935982947065e-17 0 rpy=0 0 3.141592653589793
- joint joint_body_leg_hip_4: limit lower=-0.9599310885968813 upper=0.9599310885968813 effort=12 velocity=12.0 -> lower=-0.7853981633974483 upper=0.7853981633974483 effort=45; origin xyz=-0.1093750000000001 -0.18944305707784592 0 rpy=0 0 4.1887902047863905 -> xyz=-0.10000000000000009 -0.1732050807568877 0 rpy=0 0 4.1887902047863905
- joint joint_body_leg_hip_5: limit lower=-0.9599310885968813 upper=0.9599310885968813 effort=12 velocity=12.0 -> lower=-0.7853981633974483 upper=0.7853981633974483 effort=45; origin xyz=0.10937499999999986 -0.18944305707784603 0 rpy=0 0 5.235987755982988 -> xyz=0.09999999999999987 -0.1732050807568878 0 rpy=0 0 5.235987755982988
- joint joint_leg_hip_leg_upper_0: limit lower=-1.3089969389957472 upper=1.3089969389957472 effort=30 velocity=15.0 -> lower=-1.3089969389957472 upper=1.3089969389957472 effort=30
- joint joint_leg_hip_leg_upper_1: limit lower=-1.3089969389957472 upper=1.3089969389957472 effort=30 velocity=15.0 -> lower=-1.3089969389957472 upper=1.3089969389957472 effort=30
- joint joint_leg_hip_leg_upper_2: limit lower=-1.3089969389957472 upper=1.3089969389957472 effort=30 velocity=15.0 -> lower=-1.3089969389957472 upper=1.3089969389957472 effort=30
- joint joint_leg_hip_leg_upper_3: limit lower=-1.3089969389957472 upper=1.3089969389957472 effort=30 velocity=15.0 -> lower=-1.3089969389957472 upper=1.3089969389957472 effort=30
- joint joint_leg_hip_leg_upper_4: limit lower=-1.3089969389957472 upper=1.3089969389957472 effort=30 velocity=15.0 -> lower=-1.3089969389957472 upper=1.3089969389957472 effort=30
- joint joint_leg_hip_leg_upper_5: limit lower=-1.3089969389957472 upper=1.3089969389957472 effort=30 velocity=15.0 -> lower=-1.3089969389957472 upper=1.3089969389957472 effort=30
- joint joint_leg_lower_foot_0: limit lower=0 upper=0 effort=0 velocity=0 -> lower=0 upper=0 effort=0
- joint joint_leg_lower_foot_1: limit lower=0 upper=0 effort=0 velocity=0 -> lower=0 upper=0 effort=0
- joint joint_leg_lower_foot_2: limit lower=0 upper=0 effort=0 velocity=0 -> lower=0 upper=0 effort=0
- joint joint_leg_lower_foot_3: limit lower=0 upper=0 effort=0 velocity=0 -> lower=0 upper=0 effort=0
- joint joint_leg_lower_foot_4: limit lower=0 upper=0 effort=0 velocity=0 -> lower=0 upper=0 effort=0
- joint joint_leg_lower_foot_5: limit lower=0 upper=0 effort=0 velocity=0 -> lower=0 upper=0 effort=0
- joint joint_leg_middle_leg_lower_0: limit lower=-1.5707963267948966 upper=0.7853981633974483 effort=11 velocity=15.0 -> lower=-1.5707963267948966 upper=-0.08726646259971647 effort=11
- joint joint_leg_middle_leg_lower_1: limit lower=-1.5707963267948966 upper=0.7853981633974483 effort=11 velocity=15.0 -> lower=-1.5707963267948966 upper=-0.08726646259971647 effort=11
- joint joint_leg_middle_leg_lower_2: limit lower=-1.5707963267948966 upper=0.7853981633974483 effort=11 velocity=15.0 -> lower=-1.5707963267948966 upper=-0.08726646259971647 effort=11
- joint joint_leg_middle_leg_lower_3: limit lower=-1.5707963267948966 upper=0.7853981633974483 effort=11 velocity=15.0 -> lower=-1.5707963267948966 upper=-0.08726646259971647 effort=11
- joint joint_leg_middle_leg_lower_4: limit lower=-1.5707963267948966 upper=0.7853981633974483 effort=11 velocity=15.0 -> lower=-1.5707963267948966 upper=-0.08726646259971647 effort=11
- joint joint_leg_middle_leg_lower_5: limit lower=-1.5707963267948966 upper=0.7853981633974483 effort=11 velocity=15.0 -> lower=-1.5707963267948966 upper=-0.08726646259971647 effort=11
- joint joint_leg_upper_leg_middle_0: limit lower=-1.5707963267948966 upper=0.3490658503988659 effort=22 velocity=15.0 -> lower=-1.5707963267948966 upper=-0.08726646259971647 effort=22
- joint joint_leg_upper_leg_middle_1: limit lower=-1.5707963267948966 upper=0.3490658503988659 effort=22 velocity=15.0 -> lower=-1.5707963267948966 upper=-0.08726646259971647 effort=22
- joint joint_leg_upper_leg_middle_2: limit lower=-1.5707963267948966 upper=0.3490658503988659 effort=22 velocity=15.0 -> lower=-1.5707963267948966 upper=-0.08726646259971647 effort=22
- joint joint_leg_upper_leg_middle_3: limit lower=-1.5707963267948966 upper=0.3490658503988659 effort=22 velocity=15.0 -> lower=-1.5707963267948966 upper=-0.08726646259971647 effort=22
- joint joint_leg_upper_leg_middle_4: limit lower=-1.5707963267948966 upper=0.3490658503988659 effort=22 velocity=15.0 -> lower=-1.5707963267948966 upper=-0.08726646259971647 effort=22
- joint joint_leg_upper_leg_middle_5: limit lower=-1.5707963267948966 upper=0.3490658503988659 effort=22 velocity=15.0 -> lower=-1.5707963267948966 upper=-0.08726646259971647 effort=22
