Commit message: Brand new robot

File: SpiderBot/spider.urdf (robot description, URDF)
Before this commit: robot blocky_spider, 31 links, 30 joints
Links:
- link body: mass 21.991149 -> 12.566371
- link leg_hip_0: mass 0.109375 -> 0.021875; geometry collision box size=0.035 0.025 0.025; visual box size=0.035 0.025 0.025
- link leg_hip_1: mass 0.109375 -> 0.021875; geometry collision box size=0.035 0.025 0.025; visual box size=0.035 0.025 0.025
- link leg_hip_2: mass 0.109375 -> 0.021875; geometry collision box size=0.035 0.025 0.025; visual box size=0.035 0.025 0.025
- link leg_hip_3: mass 0.109375 -> 0.021875; geometry collision box size=0.035 0.025 0.025; visual box size=0.035 0.025 0.025
- link leg_hip_4: mass 0.109375 -> 0.021875; geometry collision box size=0.035 0.025 0.025; visual box size=0.035 0.025 0.025
- link leg_hip_5: mass 0.109375 -> 0.021875; geometry collision box size=0.035 0.025 0.025; visual box size=0.035 0.025 0.025
- link leg_lower_0: mass 0.765625 -> 0.140625; geometry collision box size=0.225 0.025 0.025; visual box size=0.225 0.025 0.025
- link leg_lower_1: mass 0.765625 -> 0.140625; geometry collision box size=0.225 0.025 0.025; visual box size=0.225 0.025 0.025
- link leg_lower_2: mass 0.765625 -> 0.140625; geometry collision box size=0.225 0.025 0.025; visual box size=0.225 0.025 0.025
- link leg_lower_3: mass 0.765625 -> 0.140625; geometry collision box size=0.225 0.025 0.025; visual box size=0.225 0.025 0.025
- link leg_lower_4: mass 0.765625 -> 0.140625; geometry collision box size=0.225 0.025 0.025; visual box size=0.225 0.025 0.025
- link leg_lower_5: mass 0.765625 -> 0.140625; geometry collision box size=0.225 0.025 0.025; visual box size=0.225 0.025 0.025
- link leg_middle_0: mass 0.765625 -> 0.156250; geometry collision box size=0.25 0.025 0.025; visual box size=0.25 0.025 0.025
- link leg_middle_1: mass 0.765625 -> 0.156250; geometry collision box size=0.25 0.025 0.025; visual box size=0.25 0.025 0.025
- link leg_middle_2: mass 0.765625 -> 0.156250; geometry collision box size=0.25 0.025 0.025; visual box size=0.25 0.025 0.025
- link leg_middle_3: mass 0.765625 -> 0.156250; geometry collision box size=0.25 0.025 0.025; visual box size=0.25 0.025 0.025
- link leg_middle_4: mass 0.765625 -> 0.156250; geometry collision box size=0.25 0.025 0.025; visual box size=0.25 0.025 0.025
- link leg_middle_5: mass 0.765625 -> 0.156250; geometry collision box size=0.25 0.025 0.025; visual box size=0.25 0.025 0.025
- link leg_upper_0: mass 0.546875 -> 0.140625; geometry collision box size=0.225 0.025 0.025; visual box size=0.225 0.025 0.025
- link leg_upper_1: mass 0.546875 -> 0.140625; geometry collision box size=0.225 0.025 0.025; visual box size=0.225 0.025 0.025
- link leg_upper_2: mass 0.546875 -> 0.140625; geometry collision box size=0.225 0.025 0.025; visual box size=0.225 0.025 0.025
- link leg_upper_3: mass 0.546875 -> 0.140625; geometry collision box size=0.225 0.025 0.025; visual box size=0.225 0.025 0.025
- link leg_upper_4: mass 0.546875 -> 0.140625; geometry collision box size=0.225 0.025 0.025; visual box size=0.225 0.025 0.025
- link leg_upper_5: mass 0.546875 -> 0.140625; geometry collision box size=0.225 0.025 0.025; visual box size=0.225 0.025 0.025
Joints:
- joint joint_body_leg_hip_0: limit lower=-0.7853981633974483 upper=0.7853981633974483 effort=45 -> lower=-0.7853981633974483 upper=0.7853981633974483 effort=95
- joint joint_body_leg_hip_1: limit lower=-0.7853981633974483 upper=0.7853981633974483 effort=45 -> lower=-0.7853981633974483 upper=0.7853981633974483 effort=95
- joint joint_body_leg_hip_2: limit lower=-0.7853981633974483 upper=0.7853981633974483 effort=45 -> lower=-0.7853981633974483 upper=0.7853981633974483 effort=95
- joint joint_body_leg_hip_3: limit lower=-0.7853981633974483 upper=0.7853981633974483 effort=45 -> lower=-0.7853981633974483 upper=0.7853981633974483 effort=95
- joint joint_body_leg_hip_4: limit lower=-0.7853981633974483 upper=0.7853981633974483 effort=45 -> lower=-0.7853981633974483 upper=0.7853981633974483 effort=95
- joint joint_body_leg_hip_5: limit lower=-0.7853981633974483 upper=0.7853981633974483 effort=45 -> lower=-0.7853981633974483 upper=0.7853981633974483 effort=95
- joint joint_leg_hip_leg_upper_0: limit lower=-1.3089969389957472 upper=1.3089969389957472 effort=30 -> lower=-0.2617993877991494 upper=1.0471975511965976 effort=75; origin xyz=0.025 0 0 rpy=0 0 0.0 -> xyz=0.035 0 0 rpy=0 0 0.0
- joint joint_leg_hip_leg_upper_1: limit lower=-1.3089969389957472 upper=1.3089969389957472 effort=30 -> lower=-0.2617993877991494 upper=1.0471975511965976 effort=75; origin xyz=0.025 0 0 rpy=0 0 0.0 -> xyz=0.035 0 0 rpy=0 0 0.0
- joint joint_leg_hip_leg_upper_2: limit lower=-1.3089969389957472 upper=1.3089969389957472 effort=30 -> lower=-0.2617993877991494 upper=1.0471975511965976 effort=75; origin xyz=0.025 0 0 rpy=0 0 0.0 -> xyz=0.035 0 0 rpy=0 0 0.0
- joint joint_leg_hip_leg_upper_3: limit lower=-1.3089969389957472 upper=1.3089969389957472 effort=30 -> lower=-0.2617993877991494 upper=1.0471975511965976 effort=75; origin xyz=0.025 0 0 rpy=0 0 0.0 -> xyz=0.035 0 0 rpy=0 0 0.0
- joint joint_leg_hip_leg_upper_4: limit lower=-1.3089969389957472 upper=1.3089969389957472 effort=30 -> lower=-0.2617993877991494 upper=1.0471975511965976 effort=75; origin xyz=0.025 0 0 rpy=0 0 0.0 -> xyz=0.035 0 0 rpy=0 0 0.0
- joint joint_leg_hip_leg_upper_5: limit lower=-1.3089969389957472 upper=1.3089969389957472 effort=30 -> lower=-0.2617993877991494 upper=1.0471975511965976 effort=75; origin xyz=0.025 0 0 rpy=0 0 0.0 -> xyz=0.035 0 0 rpy=0 0 0.0
- joint joint_leg_lower_foot_0: origin xyz=0.175 0 0 rpy=0 0 0 -> xyz=0.225 0 0 rpy=0 0 0
- joint joint_leg_lower_foot_1: origin xyz=0.175 0 0 rpy=0 0 0 -> xyz=0.225 0 0 rpy=0 0 0
- joint joint_leg_lower_foot_2: origin xyz=0.175 0 0 rpy=0 0 0 -> xyz=0.225 0 0 rpy=0 0 0
- joint joint_leg_lower_foot_3: origin xyz=0.175 0 0 rpy=0 0 0 -> xyz=0.225 0 0 rpy=0 0 0
- joint joint_leg_lower_foot_4: origin xyz=0.175 0 0 rpy=0 0 0 -> xyz=0.225 0 0 rpy=0 0 0
- joint joint_leg_lower_foot_5: origin xyz=0.175 0 0 rpy=0 0 0 -> xyz=0.225 0 0 rpy=0 0 0
- joint joint_leg_middle_leg_lower_0: limit lower=-1.5707963267948966 upper=-0.08726646259971647 effort=11 -> lower=-1.4835298641951802 upper=-0.08726646259971647 effort=65; origin xyz=0.175 0 0 rpy=0 0 0.0 -> xyz=0.25 0 0 rpy=0 0 0.0
- joint joint_leg_middle_leg_lower_1: limit lower=-1.5707963267948966 upper=-0.08726646259971647 effort=11 -> lower=-1.4835298641951802 upper=-0.08726646259971647 effort=65; origin xyz=0.175 0 0 rpy=0 0 0.0 -> xyz=0.25 0 0 rpy=0 0 0.0
- joint joint_leg_middle_leg_lower_2: limit lower=-1.5707963267948966 upper=-0.08726646259971647 effort=11 -> lower=-1.4835298641951802 upper=-0.08726646259971647 effort=65; origin xyz=0.175 0 0 rpy=0 0 0.0 -> xyz=0.25 0 0 rpy=0 0 0.0
- joint joint_leg_middle_leg_lower_3: limit lower=-1.5707963267948966 upper=-0.08726646259971647 effort=11 -> lower=-1.4835298641951802 upper=-0.08726646259971647 effort=65; origin xyz=0.175 0 0 rpy=0 0 0.0 -> xyz=0.25 0 0 rpy=0 0 0.0
- joint joint_leg_middle_leg_lower_4: limit lower=-1.5707963267948966 upper=-0.08726646259971647 effort=11 -> lower=-1.4835298641951802 upper=-0.08726646259971647 effort=65; origin xyz=0.175 0 0 rpy=0 0 0.0 -> xyz=0.25 0 0 rpy=0 0 0.0
- joint joint_leg_middle_leg_lower_5: limit lower=-1.5707963267948966 upper=-0.08726646259971647 effort=11 -> lower=-1.4835298641951802 upper=-0.08726646259971647 effort=65; origin xyz=0.175 0 0 rpy=0 0 0.0 -> xyz=0.25 0 0 rpy=0 0 0.0
- joint joint_leg_upper_leg_middle_0: limit lower=-1.5707963267948966 upper=-0.08726646259971647 effort=22 -> lower=-1.8325957145940461 upper=-0.6108652381980153 effort=115; origin xyz=0.125 0 0 rpy=0 0 0.0 -> xyz=0.225 0 0 rpy=0 0 0.0
- joint joint_leg_upper_leg_middle_1: limit lower=-1.5707963267948966 upper=-0.08726646259971647 effort=22 -> lower=-1.8325957145940461 upper=-0.6108652381980153 effort=115; origin xyz=0.125 0 0 rpy=0 0 0.0 -> xyz=0.225 0 0 rpy=0 0 0.0
- joint joint_leg_upper_leg_middle_2: limit lower=-1.5707963267948966 upper=-0.08726646259971647 effort=22 -> lower=-1.8325957145940461 upper=-0.6108652381980153 effort=115; origin xyz=0.125 0 0 rpy=0 0 0.0 -> xyz=0.225 0 0 rpy=0 0 0.0
- joint joint_leg_upper_leg_middle_3: limit lower=-1.5707963267948966 upper=-0.08726646259971647 effort=22 -> lower=-1.8325957145940461 upper=-0.6108652381980153 effort=115; origin xyz=0.125 0 0 rpy=0 0 0.0 -> xyz=0.225 0 0 rpy=0 0 0.0
- joint joint_leg_upper_leg_middle_4: limit lower=-1.5707963267948966 upper=-0.08726646259971647 effort=22 -> lower=-1.8325957145940461 upper=-0.6108652381980153 effort=115; origin xyz=0.125 0 0 rpy=0 0 0.0 -> xyz=0.225 0 0 rpy=0 0 0.0
- joint joint_leg_upper_leg_middle_5: limit lower=-1.5707963267948966 upper=-0.08726646259971647 effort=22 -> lower=-1.8325957145940461 upper=-0.6108652381980153 effort=115; origin xyz=0.125 0 0 rpy=0 0 0.0 -> xyz=0.225 0 0 rpy=0 0 0.0
