Commit message: Trying to make new robot

File: SpiderBotAIProject/source/SpiderBotAIProject/SpiderBotAIProject/assets/spider_robot/urdf/spider_robot.urdf (robot description, URDF)
Before this commit: robot spider_robot, 25 links, 24 joints
Links:
- link base_link: geometry collision mesh filename=../meshes/collision/body_collision.stl scale=1 1 1; visual mesh filename=../meshes/visual/body_visual.obj scale=1 1 1
- link leg_01_inner_link: geometry collision mesh filename=../meshes/collision/leg_inner_collision.stl scale=1 1 1; visual mesh filename=../meshes/visual/leg_inner_visual.obj scale=1 1 1
- link leg_01_middle_link: geometry collision mesh filename=../meshes/collision/leg_middle_collision.stl scale=1 1 1; visual mesh filename=../meshes/visual/leg_middle_visual.obj scale=1 1 1
- link leg_01_outer_link: geometry collision mesh filename=../meshes/collision/leg_outer_collision.stl scale=1 1 1; visual mesh filename=../meshes/visual/leg_outer_visual.obj scale=1 1 1
- link leg_01_shoulder_link: geometry collision mesh filename=../meshes/collision/shoulder_collision.stl scale=1 1 1; visual mesh filename=../meshes/visual/shoulder_visual.obj scale=1 1 1
- link leg_02_inner_link: geometry collision mesh filename=../meshes/collision/leg_inner_collision.stl scale=1 1 1; visual mesh filename=../meshes/visual/leg_inner_visual.obj scale=1 1 1
- link leg_02_middle_link: geometry collision mesh filename=../meshes/collision/leg_middle_collision.stl scale=1 1 1; visual mesh filename=../meshes/visual/leg_middle_visual.obj scale=1 1 1
- link leg_02_outer_link: geometry collision mesh filename=../meshes/collision/leg_outer_collision.stl scale=1 1 1; visual mesh filename=../meshes/visual/leg_outer_visual.obj scale=1 1 1
- link leg_02_shoulder_link: geometry collision mesh filename=../meshes/collision/shoulder_collision.stl scale=1 1 1; visual mesh filename=../meshes/visual/shoulder_visual.obj scale=1 1 1
- link leg_03_inner_link: geometry collision mesh filename=../meshes/collision/leg_inner_collision.stl scale=1 1 1; visual mesh filename=../meshes/visual/leg_inner_visual.obj scale=1 1 1
- link leg_03_middle_link: geometry collision mesh filename=../meshes/collision/leg_middle_collision.stl scale=1 1 1; visual mesh filename=../meshes/visual/leg_middle_visual.obj scale=1 1 1
- link leg_03_outer_link: geometry collision mesh filename=../meshes/collision/leg_outer_collision.stl scale=1 1 1; visual mesh filename=../meshes/visual/leg_outer_visual.obj scale=1 1 1
- link leg_03_shoulder_link: geometry collision mesh filename=../meshes/collision/shoulder_collision.stl scale=1 1 1; visual mesh filename=../meshes/visual/shoulder_visual.obj scale=1 1 1
- link leg_04_inner_link: geometry collision mesh filename=../meshes/collision/leg_inner_collision.stl scale=1 1 1; visual mesh filename=../meshes/visual/leg_inner_visual.obj scale=1 1 1
- link leg_04_middle_link: geometry collision mesh filename=../meshes/collision/leg_middle_collision.stl scale=1 1 1; visual mesh filename=../meshes/visual/leg_middle_visual.obj scale=1 1 1
- link leg_04_outer_link: geometry collision mesh filename=../meshes/collision/leg_outer_collision.stl scale=1 1 1; visual mesh filename=../meshes/visual/leg_outer_visual.obj scale=1 1 1
- link leg_04_shoulder_link: geometry collision mesh filename=../meshes/collision/shoulder_collision.stl scale=1 1 1; visual mesh filename=../meshes/visual/shoulder_visual.obj scale=1 1 1
- link leg_05_inner_link: geometry collision mesh filename=../meshes/collision/leg_inner_collision.stl scale=1 1 1; visual mesh filename=../meshes/visual/leg_inner_visual.obj scale=1 1 1
- link leg_05_middle_link: geometry collision mesh filename=../meshes/collision/leg_middle_collision.stl scale=1 1 1; visual mesh filename=../meshes/visual/leg_middle_visual.obj scale=1 1 1
- link leg_05_outer_link: geometry collision mesh filename=../meshes/collision/leg_outer_collision.stl scale=1 1 1; visual mesh filename=../meshes/visual/leg_outer_visual.obj scale=1 1 1
- link leg_05_shoulder_link: geometry collision mesh filename=../meshes/collision/shoulder_collision.stl scale=1 1 1; visual mesh filename=../meshes/visual/shoulder_visual.obj scale=1 1 1
- link leg_06_inner_link: geometry collision mesh filename=../meshes/collision/leg_inner_collision.stl scale=1 1 1; visual mesh filename=../meshes/visual/leg_inner_visual.obj scale=1 1 1
- link leg_06_middle_link: geometry collision mesh filename=../meshes/collision/leg_middle_collision.stl scale=1 1 1; visual mesh filename=../meshes/visual/leg_middle_visual.obj scale=1 1 1
- link leg_06_outer_link: geometry collision mesh filename=../meshes/collision/leg_outer_collision.stl scale=1 1 1; visual mesh filename=../meshes/visual/leg_outer_visual.obj scale=1 1 1
- link leg_06_shoulder_link: geometry collision mesh filename=../meshes/collision/shoulder_collision.stl scale=1 1 1; visual mesh filename=../meshes/visual/shoulder_visual.obj scale=1 1 1
Joints:
- joint leg_05_shoulder_yaw_joint: origin xyz=-0.12299100000000011 -0.21302666087370375 0.081401 rpy=0 0 4.1887902047863905 -> xyz=-0.12299100000000011 -0.21302666087370373 0.081401 rpy=0 0 4.1887902047863905

Commit message: working on adding foot on robot

File: SpiderBotAIProject/source/SpiderBotAIProject/SpiderBotAIProject/assets/spider_robot/urdf/spider_robot.urdf (robot description, URDF)
Before this commit: robot spider_robot, 25 links, 24 joints
Links:
- added link leg_01_foot_link, mass 0.05; collision mesh filename=../meshes/collision/foot_collision.stl scale=1 1 1; visual mesh filename=../meshes/visual/foot_visual.obj scale=1 1 1
- added link leg_02_foot_link, mass 0.05; collision mesh filename=../meshes/collision/foot_collision.stl scale=1 1 1; visual mesh filename=../meshes/visual/foot_visual.obj scale=1 1 1
- added link leg_03_foot_link, mass 0.05; collision mesh filename=../meshes/collision/foot_collision.stl scale=1 1 1; visual mesh filename=../meshes/visual/foot_visual.obj scale=1 1 1
- added link leg_04_foot_link, mass 0.05; collision mesh filename=../meshes/collision/foot_collision.stl scale=1 1 1; visual mesh filename=../meshes/visual/foot_visual.obj scale=1 1 1
- added link leg_05_foot_link, mass 0.05; collision mesh filename=../meshes/collision/foot_collision.stl scale=1 1 1; visual mesh filename=../meshes/visual/foot_visual.obj scale=1 1 1
- added link leg_06_foot_link, mass 0.05; collision mesh filename=../meshes/collision/foot_collision.stl scale=1 1 1; visual mesh filename=../meshes/visual/foot_visual.obj scale=1 1 1
Joints:
- added joint leg_01_foot_fixed_joint: type fixed, parent leg_01_outer_link, child leg_01_foot_link, origin xyz=0.386244 0.016215 -0.000162 rpy=0 0 0
- added joint leg_02_foot_fixed_joint: type fixed, parent leg_02_outer_link, child leg_02_foot_link, origin xyz=0.386244 0.016215 -0.000162 rpy=0 0 0
- added joint leg_03_foot_fixed_joint: type fixed, parent leg_03_outer_link, child leg_03_foot_link, origin xyz=0.386244 0.016215 -0.000162 rpy=0 0 0
- added joint leg_04_foot_fixed_joint: type fixed, parent leg_04_outer_link, child leg_04_foot_link, origin xyz=0.386244 0.016215 -0.000162 rpy=0 0 0
- added joint leg_05_foot_fixed_joint: type fixed, parent leg_05_outer_link, child leg_05_foot_link, origin xyz=0.386244 0.016215 -0.000162 rpy=0 0 0
- added joint leg_06_foot_fixed_joint: type fixed, parent leg_06_outer_link, child leg_06_foot_link, origin xyz=0.386244 0.016215 -0.000162 rpy=0 0 0

File: SpiderBotAIProject/source/SpiderBotAIProject/SpiderBotAIProject/assets/spider_robot/urdf/spider_robot_leg_macro.xacro (robot description, xacro)
@@ -6,4 +6,5 @@
   <xacro:property name="middle_mass" value="0.18"/>
   <xacro:property name="outer_mass" value="0.16"/>
+  <xacro:property name="foot_mass" value="0.05"/>
   <xacro:property name="body_size_x" value="0.576834"/>
   <xacro:property name="body_size_y" value="0.510792"/>
@@ -21,4 +22,7 @@
   <xacro:property name="outer_size_y" value="0.088318"/>
   <xacro:property name="outer_size_z" value="0.097835"/>
+  <xacro:property name="foot_size_x" value="0.15"/>
+  <xacro:property name="foot_size_y" value="0.06"/>
+  <xacro:property name="foot_size_z" value="0.06"/>
   <xacro:property name="body_inertial_xyz" value="0 0 0.006181"/>
   <xacro:property name="shoulder_inertial_xyz" value="0.048902 0 0.032601"/>
@@ -26,4 +30,5 @@
   <xacro:property name="middle_inertial_xyz" value="0.22168 -0.0163 0"/>
   <xacro:property name="outer_inertial_xyz" value="0.226796 0.01611 -0.000166"/>
+  <xacro:property name="foot_inertial_xyz" value="0.075 0.008 0"/>
   <xacro:property name="base_to_shoulder_x" value="0.245982"/>
   <xacro:property name="base_to_shoulder_z" value="0.081401"/>
@@ -31,4 +36,5 @@
   <xacro:property name="inner_to_middle_xyz" value="0.443974 0 0"/>
   <xacro:property name="middle_to_outer_xyz" value="0.443098 0 0"/>
+  <xacro:property name="outer_to_foot_xyz" value="0.386244 0.016215 -0.000162"/>
   <xacro:property name="shoulder_joint_lower" value="-1.5708"/>
   <xacro:property name="shoulder_joint_upper" value="1.5708"/>
@@ -163,4 +169,18 @@
       <dynamics damping="${joint_damping}" friction="${joint_friction}"/>
     </joint>
+    <xacro:mesh_link
+      name="${prefix}_foot_link"
+      visual_mesh="foot_visual.obj"
+      collision_mesh="foot_collision.stl"
+      mass="${foot_mass}"
+      size_x="${foot_size_x}"
+      size_y="${foot_size_y}"
+      size_z="${foot_size_z}"
+      inertial_xyz="${foot_inertial_xyz}"/>
+    <joint name="${prefix}_foot_fixed_joint" type="fixed">
+      <origin xyz="${outer_to_foot_xyz}" rpy="0 0 0"/>
+      <parent link="${prefix}_outer_link"/>
+      <child link="${prefix}_foot_link"/>
+    </joint>
   </xacro:macro>
 </robot>
